Commit message: add license

File: cuboid_description/urdf/sensors/pico_flexx_gazebo.urdf.xacro (robot description, xacro)
@@ -1,8 +1,8 @@
 <?xml version="1.0"?>
 <robot xmlns:xacro="http://www.ros.org/wiki/xacro">
-  <!-- Microsoft Kinect / ASUS Xtion PRO Live for simulation -->
+  <!-- picoflexx for simulation -->
   <xacro:macro name="cuboid_sim_pmd_sensor" params="name">
-  <gazebo reference="${name}_link">
-    <material>Gazebo/FlatBlack</material>
+    <gazebo reference="${name}_link">
+      <material>Gazebo/FlatBlack</material>
       <sensor type="depth" name="camera">
         <always_on>true</always_on>
